Commit message: Rotate camera 90 degrees

File: neato_robot/neato_description/urdf/neato.urdf.xacro (robot description, xacro)
@@ -11,5 +11,6 @@
   <!-- neato -->
   <xacro:macro name="neato">
-	  <xacro:property name="camera_link" value="0.05" />
+	  <xacro:property name="camera_size" value="0.05" />
+    <xacro:property name="camera_length" value="0.1" />
     <link name="base_footprint"/>
     <joint name="base_joint" type="fixed">
@@ -243,5 +244,5 @@
   <joint name="camera_joint" type="fixed">
     <axis xyz="0 1 0" />
-    <origin xyz="-0.1 0 0.25" rpy="0 0 0"/>
+    <origin xyz="-0.1 0 0.25" rpy="0 0 ${M_PI/2}"/>
     <parent link="base_link"/>
     <child link="camera_link"/>
@@ -251,5 +252,5 @@
       <origin xyz="0 0 0" rpy="0 0 0"/>
       <geometry>
-    <box size="${camera_link} ${camera_link} ${camera_link}"/>
+    <box size="${camera_length} ${camera_size} ${camera_size}"/>
       </geometry>
     </collision>
@@ -257,5 +258,5 @@
       <origin xyz="0 0 0" rpy="0 0 0"/>
       <geometry>
-    <box size="${camera_link} ${camera_link} ${camera_link}"/>
+    <box size="${camera_length} ${camera_size} ${camera_size}"/>
       </geometry>
       <material name="red"/>
